File: 04.PCB/副机 插座 v0.3.brd (EAGLE design)
At the start: 36.8 x 45.4 mm, 26 parts, among them Y2 RESONATORSMD

Commit message: 更新了几个新pcb
更新了几个新pcb
Parts:
- BT13X: value BT136 -> BT138-H; device PKJ:TO252 -> triac:TO220BH
- R1, R4: device resistor:0204/7 -> MY3:1206
- moved U$2 8.99 mm to (8.89, 4.13)
- moved R4 7.96 mm to (15.2, 5.08)
- moved U$1 5.97 mm to (22.5, 4.13)
- moved C2 5.24 mm to (21.0, 6.99)
- moved BT13X 4.24 mm to (16.2, 12.1)
- moved R1 3.38 mm to (26.0, 7.94), turned to 90 degrees
- moved KEY 0.90 mm to (6.35, 23.2)
- moved MOC3041 0.71 mm to (32.1, 12.1)
- moved C13 0.32 mm to (17.1, 21.3)
- moved C14 0.32 mm to (20.3, 21.3)
Connections:
- net IN: now also BT13X.T2; no longer BT13X.3
- net N$2: now also BT13X.G; no longer BT13X.2
- net OUT: now also BT13X.T1; no longer BT13X.1
Routing:
- net OUT: track 11.1 -> 6.35 mm, vias 7 -> 1
- net N$2: track 15.6 -> 11.2 mm
- net N$6: track 1.59 -> 3.31 mm
- net P1: track 7.10 -> 7.86 mm
- net IN: track 30.1 -> 30.5 mm, vias 10 -> 1
- net GND: vias 36 -> 35
