File: 04.PCB/主机 v0.2.brd (EAGLE design)
At the start: 50.5 x 49.5 mm, 59 parts, among them IC1 ASM1117, IC2 ATMEGA644A, IC3 ASM1117, X1 J1011F, Y1 25M, Y2 RESONATORSMD

Commit message: 更新
Other:
- outline, holes or cut-outs redrawn
Changed lines of the file:
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@@
 <wire x1="0.23495" y1="2.1209" x2="2.13995" y2="0.2159" width="0.3048" layer="20" curve="90"/>
 <wire x1="0.23495" y1="48.0441" x2="0.23495" y2="24.0919" width="0.3048" layer="20"/>
-<wire x1="0.23495" y1="2.1209" x2="0.23495" y2="12.1412" width="0.3048" layer="20"/>
+<wire x1="0.23495" y1="2.1209" x2="0.23495" y2="7.0612" width="0.3048" layer="20"/>
 <wire x1="27.78125" y1="13.97" x2="32.22625" y2="13.97" width="0.254" layer="21"/>
 <wire x1="32.22625" y1="13.97" x2="32.22625" y2="14.605" width="0.254" layer="21"/>
@@
 <wire x1="1.55575" y1="22.6187" x2="1.55575" y2="17.2085" width="0.3048" layer="20"/>
 <wire x1="1.55575" y1="17.2085" x2="0.20955" y2="15.8623" width="0.3048" layer="20"/>
-<wire x1="0.20955" y1="15.8623" x2="0.20955" y2="11.7983" width="0.3048" layer="20"/>
+<wire x1="0.20955" y1="15.8623" x2="0.20955" y2="14.44625" width="0.3048" layer="20"/>
+<wire x1="0.20955" y1="14.44625" x2="0.635" y2="14.44625" width="0.3048" layer="20"/>
+<wire x1="0.635" y1="14.44625" x2="0.635" y2="7.14375" width="0.3048" layer="20"/>
+<wire x1="0.635" y1="7.14375" x2="0.3175" y2="7.14375" width="0.3048" layer="20"/>
 <wire x1="50.52695" y1="21.7043" x2="49.54905" y2="20.7264" width="0.3048" layer="20"/>
 <wire x1="49.54905" y1="20.7264" x2="49.54905" y2="17.8054" width="0.3048" layer="20"/>
@@
 <via x="3.96875" y="5.87375" extent="1-16" drill="0.3048"/>
 <via x="4.92125" y="5.87375" extent="1-16" drill="0.3048"/>
-<via x="1.07315" y="12.51585" extent="1-16" drill="0.3048"/>
-<via x="1.07315" y="11.56335" extent="1-16" drill="0.3048"/>
-<via x="1.07315" y="10.61085" extent="1-16" drill="0.3048"/>
-<via x="1.07315" y="9.65835" extent="1-16" drill="0.3048"/>
-<via x="1.07315" y="8.70585" extent="1-16" drill="0.3048"/>
+<via x="1.8669" y="12.51585" extent="1-16" drill="0.3048"/>
+<via x="1.8669" y="11.56335" extent="1-16" drill="0.3048"/>
+<via x="1.8669" y="10.61085" extent="1-16" drill="0.3048"/>
+<via x="1.8669" y="9.65835" extent="1-16" drill="0.3048"/>
+<via x="1.8669" y="8.70585" extent="1-16" drill="0.3048"/>
 <contactref element="C17" pad="1"/>
 <contactref element="C18" pad="1"/>
@@
 <via x="28.2575" y="47.625" extent="1-16" drill="0.3048"/>
 <via x="28.2575" y="46.83125" extent="1-16" drill="0.3048"/>
-<via x="24.60625" y="35.2425" extent="1-16" drill="0.3048"/>
-<via x="21.74875" y="38.1" extent="1-16" drill="0.3048"/>
+<via x="24.765" y="35.2425" extent="1-16" drill="0.3048"/>
+<via x="21.9075" y="38.25875" extent="1-16" drill="0.3048"/>
 <via x="28.575" y="39.0525" extent="1-16" drill="0.3048"/>
 <via x="29.845" y="39.0525" extent="1-16" drill="0.3048"/>
@@
 <contactref element="ASP" pad="7"/>
 <wire x1="21.11995" y1="42.8309" x2="19.52625" y2="41.2372" width="0.4064" layer="1"/>
-<wire x1="19.52625" y1="41.2372" x2="19.52625" y2="38.89375" width="0.4064" layer="1"/>
-<wire x1="24.28875" y1="33.17875" x2="26.908125" y2="30.559375" width="0.4064" layer="1"/>
+<wire x1="19.52625" y1="41.2372" x2="19.52625" y2="39.21125" width="0.4064" layer="1"/>
+<wire x1="24.4475" y1="33.02" x2="26.908125" y2="30.559375" width="0.4064" layer="1"/>
 <wire x1="14.418959375" y1="25.06961875" x2="14.418959375" y2="26.483959375" width="0.3556" layer="1"/>
 <wire x1="14.418959375" y1="26.483959375" x2="15.875" y2="27.94" width="0.3556" layer="1"/>
@@
 <wire x1="31.75" y1="24.4475" x2="31.75" y2="25.7175" width="0.4064" layer="16"/>
 <wire x1="31.75" y1="25.7175" x2="30.7975" y2="26.67" width="0.4064" layer="16"/>
-<wire x1="24.28875" y1="33.17875" x2="24.28875" y2="34.13125" width="0.4064" layer="1"/>
-<wire x1="24.28875" y1="34.13125" x2="19.52625" y2="38.89375" width="0.4064" layer="1"/>
+<wire x1="24.4475" y1="33.02" x2="24.4475" y2="34.29" width="0.4064" layer="1"/>
+<wire x1="24.4475" y1="34.29" x2="19.52625" y2="39.21125" width="0.4064" layer="1"/>
 </signal>
 <signal name="D12/MISO">
